File: invertercontroller.sch (KiCad schematic (older format))
At the start: 39 parts, among them P1 bat voltage, P2 12vacin, P3 temp sensor, P4 fan, P5 inretershutdownout, P6 temp shut sensor2, Q1 Q_NMOS_DGS, Q2 Q_NPN_BCE, Q3 Q_NPN_BCE, Q4 Q_NPN_BCE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

Commit message: added pdf of schematic
Parts:
- U3: footprint DIP-4 -> Opto-Devices:Optocoupler_SMD_HandSoldering_KPC357_LTV35x_PC357_SingleChannel
- fantemp1, highvolts1, lowvolts1, tempdelay1, tempshutdown1: footprint Potentiometers:Potentiometer_Trimmer-Piher-PT15-h2-5_vertical -> Potentiometers:Potentiometer_WirePads_Small
Changed lines of the file:
@@
 F 0 "fantemp1" H 1825 2170 50  0000 C CNN
 F 1 "10k" H 1825 2250 50  0000 C CNN
-F 2 "Potentiometers:Potentiometer_Trimmer-Piher-PT15-h2-5_vertical" H 1825 2250 50  0001 C CNN
+F 2 "Potentiometers:Potentiometer_WirePads_Small" H 1825 2250 50  0001 C CNN
 F 3 "" H 1825 2250 50  0000 C CNN
 	1    1825 2250
@@
 F 0 "tempdelay1" H 3375 2520 50  0000 C CNN
 F 1 "10k" H 3375 2600 50  0000 C CNN
-F 2 "Potentiometers:Potentiometer_Trimmer-Piher-PT15-h2-5_vertical" H 3375 2600 50  0001 C CNN
+F 2 "Potentiometers:Potentiometer_WirePads_Small" H 3375 2600 50  0001 C CNN
 F 3 "" H 3375 2600 50  0000 C CNN
 	1    3375 2600
@@
 F 0 "highvolts1" H 1725 4345 50  0000 C CNN
 F 1 "100k" H 1725 4425 50  0000 C CNN
-F 2 "Potentiometers:Potentiometer_Trimmer-Piher-PT15-h2-5_vertical" H 1725 4425 50  0001 C CNN
+F 2 "Potentiometers:Potentiometer_WirePads_Small" H 1725 4425 50  0001 C CNN
 F 3 "" H 1725 4425 50  0000 C CNN
 	1    1725 4425
@@
 F 0 "lowvolts1" H 1800 6020 50  0000 C CNN
 F 1 "100k" H 1800 6100 50  0000 C CNN
-F 2 "Potentiometers:Potentiometer_Trimmer-Piher-PT15-h2-5_vertical" H 1800 6100 50  0001 C CNN
+F 2 "Potentiometers:Potentiometer_WirePads_Small" H 1800 6100 50  0001 C CNN
 F 3 "" H 1800 6100 50  0000 C CNN
 	1    1800 6100
@@
 F 0 "U3" H 4575 3775 50  0000 L CNN
 F 1 "PC817" H 4775 3775 50  0000 L CNN
-F 2 "DIP-4" H 4575 3375 50  0000 L CIN
+F 2 "Opto-Devices:Optocoupler_SMD_HandSoldering_KPC357_LTV35x_PC357_SingleChannel" H 4575 3375 50  0000 L CIN
 F 3 "" H 4775 3575 50  0000 L CNN
 	1    4775 3575
@@
 F 0 "tempshutdown1" H 6650 5545 50  0000 C CNN
 F 1 "10k" H 6650 5625 50  0000 C CNN
-F 2 "Potentiometers:Potentiometer_Trimmer-Piher-PT15-h2-5_vertical" H 6650 5625 50  0001 C CNN
+F 2 "Potentiometers:Potentiometer_WirePads_Small" H 6650 5625 50  0001 C CNN
 F 3 "" H 6650 5625 50  0000 C CNN
 	1    6650 5625
